Commit message: Viewer: laptop rebuilt with the current fit (replay covers lid 95%, base 94%)
Co-Authored-By: Claude Opus 5.5 <noreply@anthropic.com>

File: docs/models/laptop_lidar/model.urdf (robot description, URDF)
Before this commit: robot laptop_lidar, 2 links, 1 joints
Joints:
- joint lid_joint: limit lower=-1.9884 upper=0.0265 effort=10 velocity=2 -> lower=-1.8613 upper=0.1638 effort=10 velocity=2

Commit message: Viewer and robot demo show the video-textured laptop; one shared texture atlas
The textured OBJ meshes share one atlas (video_tex.png, 2 MB instead of three copies).
The viewer loads them with three.js's OBJLoader; the robot scene copies the model's textures
and materials. [hidden] now beats .seg's display: flex (the Realistic/Measured switch showed
on models without SAM 3D meshes).

Co-Authored-By: Claude Opus 5.5 <noreply@anthropic.com>

File: docs/models/laptop_lidar/model.urdf (robot description, URDF)
Before this commit: robot laptop_lidar, 2 links, 1 joints
Links:
- link base: geometry collision mesh filename=meshes/base.stl; visual mesh filename=meshes/base_tex.obj
- link lid: geometry collision mesh filename=meshes/lid.stl; visual mesh filename=meshes/lid_tex.obj
