Commit message: Viewer and demo: the agent's drawer (pulls out 248 mm); demo 2:55 with a drawer scene
Co-Authored-By: Claude Opus 5.5 <noreply@anthropic.com>

File: docs/models/drawer/model.urdf (robot description, URDF)
Before this commit: robot drawer2_lidar, 2 links, 1 joints
Links:
- link base: geometry collision mesh filename=meshes/base_0.stl; collision mesh filename=meshes/base_1.stl
Joints:
- joint drawer1_joint: axis 1.00000 0.00000 0.00000 -> 1.00000 0.00000 -0.00000; limit lower=0.0000 upper=0.2530 effort=10 velocity=2 -> lower=0.0000 upper=0.2480 effort=10 velocity=2

Commit message: Viewer: each model's masses, and its joint friction with the MuJoCo release check
Robot demos re-rendered with the measured masses and friction (laptop closes to -80 of -77 deg).

Co-Authored-By: Claude Opus 5.5 <noreply@anthropic.com>

File: docs/models/drawer/model.urdf (robot description, URDF)
Before this commit: robot drawer2_lidar, 2 links, 1 joints
Links:
- link base: mass None -> 13
- link drawer1: mass None -> 2.5

File: docs/models/laptop_lidar/model.urdf (robot description, URDF)
Before this commit: robot laptop_lidar, 2 links, 1 joints
Links:
- link base: mass None -> 0.9
- link lid: mass None -> 0.5

File: docs/models/notebook/model.urdf (robot description, URDF)
Before this commit: robot notebook_2, 2 links, 1 joints
Links:
- link base: mass None -> 0.95
- link lid: mass None -> 0.45

File: docs/models/stand/model.urdf (robot description, URDF)
Before this commit: robot stand_2, 3 links, 2 joints
Links:
- link base: mass None -> 0.45
- link lower_arm: mass None -> 0.075
- link upper_arm: mass None -> 0.09

Commit message: Viewer: the drawer's front painted with its video (wood grain and handle)
Co-Authored-By: Claude Opus 5.5 <noreply@anthropic.com>

File: docs/models/drawer/model.urdf (robot description, URDF)
Before this commit: robot drawer2_lidar, 2 links, 1 joints
Links:
- link base: geometry collision mesh filename=meshes/base_0.stl; collision mesh filename=meshes/base_1.stl
- link drawer1: geometry collision mesh filename=meshes/drawer1_0.stl; collision mesh filename=meshes/drawer1_1.stl

Commit message: Viewer: the four demo models with Spark's designed visuals (Realistic) over the measured ones (Measured)
Co-Authored-By: Claude Opus 5.5 <noreply@anthropic.com>

File: docs/models/drawer/model.urdf (robot description, URDF)
Before this commit: robot drawer2_lidar, 2 links, 1 joints
Links:
- link base: geometry collision mesh filename=meshes/base_0.stl; collision mesh filename=meshes/base_1.stl
- link drawer1: geometry collision mesh filename=meshes/drawer1_0.stl; collision mesh filename=meshes/drawer1_1.stl

File: docs/models/laptop_lidar/model.urdf (robot description, URDF)
Before this commit: robot laptop_lidar, 2 links, 1 joints
Links:
- link base: geometry collision mesh filename=meshes/base.stl; visual box size=0.11500 0.07500 0.00120
- link lid: geometry collision mesh filename=meshes/lid.stl; visual box size=0.19327 0.28500 0.00120

File: docs/models/notebook/model.urdf (robot description, URDF)
Before this commit: robot notebook_2, 2 links, 1 joints
Links:
- link base: geometry collision mesh filename=meshes/base.stl; visual box size=0.03500 0.07500 0.00100
- link lid: geometry collision mesh filename=meshes/lid.stl; visual box size=0.00120 0.22000 0.11800

File: docs/models/stand/model.urdf (robot description, URDF)
Before this commit: robot stand_2, 3 links, 2 joints
Links:
- link base: geometry collision mesh filename=meshes/base.stl; visual box size=0.01400 0.01600 0.01000
- link lower_arm: geometry collision mesh filename=meshes/lower_arm.stl; visual box size=0.00894 0.01000 0.00700
- link upper_arm: geometry collision mesh filename=meshes/upper_arm.stl; visual box size=0.20861 0.01100 0.00180
