Commit message: Viewer: robot task videos for the laptop, drawer, lamp, mouse and side-view laptop; the refitted LiDAR lamp
Co-Authored-By: Claude Opus 5.5 <noreply@anthropic.com>

File: docs/models/lamp_lidar/model.urdf (robot description, URDF)
Before this commit: robot stand_lidar, 3 links, 2 joints
Links:
- link lamp_base: geometry collision mesh filename=meshes/base.stl; visual box size=0.00800 0.00800 0.00080
- link rod1: geometry collision mesh filename=meshes/rod1.stl; visual box size=0.35127 0.02400 0.00800
- link rod2: geometry collision mesh filename=meshes/rod2.stl; visual box size=0.38023 0.02400 0.00800
Joints:
- joint rod1_joint: axis 0.99891 0.00000 -0.04675 -> (none); limit lower=-0.3744 upper=0.9165 effort=10 velocity=2 -> (none); origin xyz=0.08305 0.06557 0.08146 rpy=0 0 0 -> xyz=0.08271 0.06173 0.02411 rpy=0 0 0; type revolute -> fixed
- joint rod2_joint: axis 0.07712 -0.98077 0.17927 -> 0.13633 -0.99064 -0.00714; limit lower=-0.1347 upper=1.3434 effort=10 velocity=2 -> lower=0.0326 upper=1.5515 effort=10 velocity=2; origin xyz=0.00597 0.02474 0.29137 rpy=0 0 0 -> xyz=0.00581 -0.00403 0.35116 rpy=0 0 0
