Commit message: docs/models: portable downloads for seven tabs (export_viewer.py --repack; microwave left to its owner)
model.urdf, model.xml and model.zip of airpods_lidar, drawer, lamp_lidar, laptop_lidar,
mouse_lidar, notebook and stand: OBJ twins of the URDF's STLs (Drake), MuJoCo's strippath
block, a header on how to load them, and the laptop's and lamp's base inertial frames (5 deg
off at gimbal lock) rewritten from model.xml. model.json, index.json, meshes the viewer loads
and videos are untouched; the viewer still loads (headless Chrome, laptop and drawer tabs).
scripts/check_exports.py on docs/models: 0 failures on these seven except notebook's URDF in
MuJoCo (its lid overlaps the base by 13 mm at the hinge and a URDF can't exclude that contact).

Co-Authored-By: Claude Opus 5.5 <noreply@anthropic.com>
Claude-Session: https://claude.ai/code/session_01G1sGHxozTsCqmS7N3h3a3L

File: docs/models/airpods_lidar/model.urdf (robot description, URDF)
Before this commit: robot airpods_lidar, 1 links, 0 joints
Links:
- link base: geometry collision mesh filename=meshes/static_object.obj; visual box size=0.00922 0.00180 0.00220

File: docs/models/drawer/model.urdf (robot description, URDF)
Before this commit: robot drawer2_lidar, 2 links, 1 joints
Links:
- link base: geometry collision mesh filename=meshes/base_0.obj; collision mesh filename=meshes/base_1.obj
- link drawer1: geometry collision mesh filename=meshes/drawer1_0.obj; collision mesh filename=meshes/drawer1_1.obj

File: docs/models/lamp_lidar/model.urdf (robot description, URDF)
Before this commit: robot stand_lidar, 3 links, 2 joints
Links:
- link lamp_base: geometry collision mesh filename=meshes/base.obj; visual box size=0.00800 0.00800 0.00080
- link rod1: geometry collision mesh filename=meshes/rod1.obj; visual box size=0.35127 0.02400 0.00800
- link rod2: geometry collision mesh filename=meshes/rod2.obj; visual box size=0.38023 0.02400 0.00800

File: docs/models/laptop_lidar/model.urdf (robot description, URDF)
Before this commit: robot laptop_lidar, 2 links, 1 joints
Links:
- link base: geometry collision mesh filename=meshes/base.obj; visual box size=0.11500 0.07500 0.00120
- link lid: geometry collision mesh filename=meshes/lid.obj; visual box size=0.19327 0.28500 0.00120

File: docs/models/mouse_lidar/model.urdf (robot description, URDF)
Before this commit: robot mouse_lidar, 1 links, 0 joints
Links:
- link base: geometry collision mesh filename=meshes/static_object.obj; visual mesh filename=meshes/base_sam3d.obj

File: docs/models/notebook/model.urdf (robot description, URDF)
Before this commit: robot notebook_2, 2 links, 1 joints
Links:
- link base: geometry collision mesh filename=meshes/base.obj; visual box size=0.03500 0.07500 0.00100
- link lid: geometry collision mesh filename=meshes/lid.obj; visual box size=0.00120 0.22000 0.11800

File: docs/models/stand/model.urdf (robot description, URDF)
Before this commit: robot stand_2, 3 links, 2 joints
Links:
- link base: geometry collision mesh filename=meshes/base.obj; visual box size=0.01400 0.01600 0.01000
- link lower_arm: geometry collision mesh filename=meshes/lower_arm.obj; visual box size=0.00894 0.01000 0.00700
- link upper_arm: geometry collision mesh filename=meshes/upper_arm.obj; visual box size=0.20861 0.01100 0.00180
