Commit message: Microwave tab: the completed body (front measured, depth bounded by the video, rest estimated by Muse Spark)
Exported from a copy of the published run (data/agentE/microwave_lidar) after
scripts/complete_body.py: 477 x 365 x 269 mm; the front is measured (LiDAR inside a SAM 3.1 mask
of the whole microwave), the depth lies between the cavity's back seen through the open door
(329 mm, +wall) and a wall seen behind the top (387 mm), Spark (Samsung 23 L) puts it at 365 mm;
cavity 330 x 205 x 295 mm (depth measured), body ~10 kg (estimated). Hollow carcass of boxes that
collides; the door, hinge and textures are unchanged. Replay over the video redone with the body;
the Not measured note lists every estimate; provenance says the body was completed afterwards.
CLAUDE.md: what the completion step does, its results and lessons.

Co-Authored-By: Claude Opus 5.5 <noreply@anthropic.com>
Claude-Session: https://claude.ai/code/session_01G1sGHxozTsCqmS7N3h3a3L

File: docs/models/microwave_lidar/model.urdf (robot description, URDF)
Before this commit: robot microwave_lidar, 2 links, 1 joints
Links:
- link base: mass 0.05 -> 10.2; geometry collision box size=0.029594 0.330638 0.205; collision box size=0.029594 0.330638 0.205

Commit message: Microwave base inertia from the completed body (COM and moments were the measured strip's at 10.2 kg), its downloads made portable; the viewer hands out the zip first; README: the downloads checked in MuJoCo, PyBullet, yourdfpy and Drake
Co-Authored-By: Claude Opus 5.5 <noreply@anthropic.com>
Claude-Session: https://claude.ai/code/session_01G1sGHxozTsCqmS7N3h3a3L

File: docs/models/microwave_lidar/model.urdf (robot description, URDF)
Before this commit: robot microwave_lidar, 2 links, 1 joints
Links:
- link base: geometry collision box size=0.029594 0.330638 0.205; collision box size=0.029594 0.330638 0.205
- link lid: geometry collision mesh filename=meshes/lid.obj; visual mesh filename=meshes/lid_tex.obj
